Commit message: Completion of simulator

File: xacro/msd_tunnel_dtw.xacro (robot description, xacro)
@@ -2,15 +2,15 @@
 <robot name="msd_tunnel_dtw" xmlns:xacro="http://ros.org/wiki/xacro">
   <material name="gray">
-    <color rgba="0.5 0.5 0.5 2.5"/>
+    <color rgba="0.5 0.5 0.5 1.0"/>
   </material>
   <material name="red">
-    <color rgba="1.0 0.0 0.0 2.5"/>
+    <color rgba="1.0 0.0 0.0 1.0"/>
   </material>
-  <xacro:macro name="wheel_macro" params="parent prefix xyz">
+  <xacro:macro name="drive_wheel" params="parent prefix xyz">
     <joint name="${prefix}_joint" type="continuous">
-      <origin xyz="${xyz}" rpy="${radians(-90)} 0 0"/>
+      <origin xyz="${xyz}" rpy="0 0 0"/>
       <parent link="${parent}"/>
       <child  link="${prefix}_link"/>
-      <axis xyz="0 0 1" />
+      <axis xyz="0 1 0" />
     </joint>
     <transmission name="${prefix}_trans" type="SimpleTransmission">
@@ -25,17 +25,17 @@
     <link name="${prefix}_link">
       <inertial>
-        <origin xyz="0 0 0" rpy="0 0 0"/>
-        <mass value="0.1"/>
+        <mass value="3.5"/>
         <inertia ixx="0.0001" ixy="0.0" ixz="0.0" iyy="0.0001" iyz="0.0" izz="0.0001"/>
       </inertial>
       <visual>
         <geometry>
-          <cylinder radius="0.05" length="0.02" />
+          <mesh filename="package://msd_simulator/model/meshes/msd_tunnel/drive_wheel.dae"/>
         </geometry>
         <material name="red"/>
       </visual>
       <collision>
+        <origin xyz="0 0 0" rpy="1.57 0 0"/>
         <geometry>
-          <cylinder radius="0.05" length="0.02" />
+          <cylinder radius="0.1105" length="0.076" />
         </geometry>
       </collision>
@@ -43,7 +43,40 @@
     <gazebo reference="${prefix}_link">
       <material>Gazebo/Red</material>
-      <mu1 value="2.5" />
-      <mu2 value="2.5" />
-      <kp value="50000" />
+      <mu1 value="1.0" />
+      <mu2 value="1.0" />
+      <kp value="10000000" />
+      <kd value="10" />
+    </gazebo>
+  </xacro:macro>
+  <xacro:macro name="roller" params="prefix xyz">
+    <joint name="${prefix}_joint" type="fixed">
+      <parent link="base_link"/>
+      <child  link="${prefix}_link"/>
+      <origin xyz="${xyz}" rpy="0 0 0"/>
+    </joint>
+    <link name="${prefix}_link">
+      <inertial>
+        <mass value="1.1"/>
+        <inertia ixx="0.0001" ixy="0.0" ixz="0.0" iyy="0.0001" iyz="0.0" izz="0.0001"/>
+      </inertial>
+      <visual>
+        <origin xyz="0 0 0" rpy="0 0 0" />
+        <geometry>
+          <mesh filename="package://msd_simulator/model/meshes/msd_tunnel/roller.dae" />
+        </geometry>
+      </visual>
+      <collision>
+        <origin xyz="0 0 0" rpy="1.57 0 0" />
+        <geometry>
+          <cylinder radius="0.055" length="0.076" />
+        </geometry>
+        <material name="gray" />
+      </collision>
+    </link>
+    <gazebo reference="${prefix}_link">
+      <material>Gazebo/Gray</material>
+      <mu1 value="0.1" />
+      <mu2 value="0.1" />
+      <kp value="10000000" />
       <kd value="10" />
     </gazebo>
@@ -53,10 +86,10 @@
     <parent link="base_link"/>
     <child  link="body_link"/>
-    <origin xyz="-0.07 0 0.07" rpy="0 0 0"/>
+    <origin xyz="0 0 0" rpy="0 0 0"/>
   </joint>
   <link name="body_link">
     <inertial>
       <origin xyz="0 0 0" rpy="0 0 0"/>
-      <mass value="1.0"/>
+      <mass value="182.8"/>
       <inertia ixx="0.001" ixy="0.0" ixz="0.0" iyy="0.001" iyz="0.0" izz="0.001"/>
     </inertial>
@@ -64,12 +97,11 @@
       <origin xyz="0 0 0" rpy="0 0 0" />
       <geometry>
-        <box size="0.24 0.18 0.06" />
+        <mesh filename="package://msd_simulator/model/meshes/msd_tunnel/body.dae" />
       </geometry>
-      <material name="gray" />
     </visual>
     <collision>
-      <origin xyz="0 0 0" rpy="0 0 0" />
+      <origin xyz="0 0 0.250" rpy="0 0 0" />
       <geometry>
-        <box size="0.24 0.178 0.06" />
+        <box size="0.800 0.480 0.400" />
       </geometry>
     </collision>
@@ -78,32 +110,11 @@
     <material>Gazebo/Gray</material>
   </gazebo>
-  <xacro:wheel_macro prefix="left_wheel"  parent="base_link" xyz="0 0.1 0.05"/>
-  <xacro:wheel_macro prefix="right_wheel" parent="base_link" xyz="0 -0.1 0.05"/>
-  <joint name="ball_joint" type="fixed">
-    <parent link="base_link"/>
-    <child  link="ball_link"/>
-    <origin xyz="-0.14 0 0.04" rpy="0 0 0"/>
-  </joint>
-  <link name="ball_link">
-    <visual>
-      <origin xyz="0 0 0" rpy="0 0 0" />
-      <geometry>
-        <sphere radius="0.04" />
-      </geometry>
-      <material name="gray" />
-    </visual>
-    <collision>
-      <origin xyz="0 0 0" rpy="0 0 0" />
-      <geometry>
-        <sphere radius="0.04" />
-      </geometry>
-      <material name="gray" />
-    </collision>
-  </link>
-  <gazebo reference="ball_link">
-    <material>Gazebo/Gray</material>
-    <mu1 value="0.5" />
-    <mu2 value="0.5" />
-  </gazebo>
+  <xacro:drive_wheel prefix="left_wheel"  parent="base_link" xyz="-0.2575 0.300 0.1105"/>
+  <xacro:drive_wheel prefix="right_wheel" parent="base_link" xyz="-0.2575 -0.300 0.1105"/>
+  <!-- -0.2575 -300 0.053 -->
+  <xacro:roller prefix="left_front" xyz="0.287 0.295 0.055"/>
+  <xacro:roller prefix="left_center" xyz="0.0175 0.295 0.055"/>
+  <xacro:roller prefix="right_front" xyz="0.287 -0.295 0.055"/>
+  <xacro:roller prefix="right_center" xyz="0.0175 -0.295 0.055"/>
   <gazebo>
     <plugin name="gazebo_ros_control" filename="libgazebo_ros_control.so">

Commit message: first lidar sim demo

File: xacro/msd_tunnel_dtw.xacro (robot description, xacro)
@@ -2,5 +2,5 @@
 <robot name="msd_tunnel_dtw" xmlns:xacro="http://ros.org/wiki/xacro">
   <material name="gray">
-    <color rgba="0.5 0.5 0.5 1.0"/>
+    <color rgba="0.3 0.3 0.3 1.0"/>
   </material>
   <material name="red">
@@ -71,5 +71,4 @@
           <cylinder radius="0.055" length="0.076" />
         </geometry>
-        <material name="gray" />
       </collision>
     </link>
@@ -91,5 +90,5 @@
     <inertial>
       <origin xyz="0 0 0" rpy="0 0 0"/>
-      <mass value="182.8"/>
+      <mass value="18.28"/>
       <inertia ixx="0.001" ixy="0.0" ixz="0.0" iyy="0.001" iyz="0.0" izz="0.001"/>
     </inertial>
@@ -99,4 +98,5 @@
         <mesh filename="package://msd_simulator/model/meshes/msd_tunnel/body.dae" />
       </geometry>
+      <material name="gray" />
     </visual>
     <collision>
