Commit message: create rplidar sim

File: xacro/msd_tunnel_sensor.urdf (robot description, URDF)
Before this commit: robot msd_tunnel_dtw, 9 links, 8 joints
Links:
- link rplidar_s1_link: geometry collision cylinder length=0.06 radius=0.02; visual mesh filename=package://msd_simulator/model/meshes/msd_tunnel/rplidar-s1m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
Joints:
- joint rplidar_s1_joint: origin xyz=0.4385 0 0.2121 rpy=0 0 0 -> xyz=0.4385 0 0.387 rpy=0 0 0

File: xacro/msd_tunnel_sensor.xacro (robot description, xacro)
@@ -1,4 +1,4 @@
 <?xml version="1.0"?>
-<robot name="msd_tunnel_dtw" xmlns:xacro="http://ros.org/wiki/xacro">
+<robot name="msd_tunnel_sensor" xmlns:xacro="http://ros.org/wiki/xacro">
   <material name="gray">
     <color rgba="0.3 0.3 0.3 1.0"/>
@@ -90,6 +90,9 @@
       <visual>
         <origin xyz="0 0 0" rpy="0 0 0" />
+        <!-- <geometry>
+          <cylinder radius="0.025" length="0.050" />
+        </geometry> -->
         <geometry>
-          <cylinder radius="0.02" length="0.06" />
+          <mesh filename="package://msd_simulator/model/meshes/msd_tunnel/rplidar-s1m1-r1.dae"/>
         </geometry>
         <material name="red" />
@@ -97,6 +100,9 @@
       <collision>
         <origin xyz="0 0 0" rpy="0 0 0"/>
+        <!-- <geometry>
+          <cylinder radius="0.025" length="0.050" />
+        </geometry> -->
         <geometry>
-          <cylinder radius="0.02" length="0.06" />
+          <mesh filename="package://msd_simulator/model/meshes/msd_tunnel/rplidar-s1m1-r1.dae"/>
         </geometry>
       </collision>
@@ -105,21 +111,22 @@
       <material>Gazebo/Red</material>
       <sensor type="ray" name="${prefix}">
-        <pose>0 0 0 0 0 0</pose>
+        <origin xyz="0 0 0.037" rpy="0 0 0"/>
         <visualize>true</visualize>
         <update_rate>10</update_rate>
         <ray>
           <scan>
+            <origin xyz="0 0 0.037" rpy="0 0 0"/>
             <horizontal>
-              <samples>400</samples>
+              <samples>9200</samples> <!-- per second 9200 -->
               <resolution>1</resolution>
-              <min_angle>${radians(-90)}</min_angle>
-              <max_angle>${radians( 90)}</max_angle>
+              <min_angle>-3.14</min_angle>
+              <max_angle>3.14</max_angle> <!-- 360 degree = 3.14-->
             </horizontal>
           </scan>
-          <range>
-            <min>0.10</min>
-            <max>20.0</max>
-            <resolution>0.01</resolution>
-          </range>
+            <range>
+              <min>0.10</min>
+              <max>40.0</max>
+              <resolution>0.01</resolution> <!-- ? -->
+            </range>
           <noise>
             <type>gaussian</type>
@@ -170,8 +177,9 @@
   <xacro:roller prefix="right_front" xyz="0.287 -0.295 0.055"/>
   <xacro:roller prefix="right_center" xyz="0.0175 -0.295 0.055"/>
-  <xacro:laser_macro prefix="rplidar_s1" parent="base_link" xyz="0.4385 0 0.2121"/>
+  <xacro:laser_macro prefix="rplidar_s1" parent="base_link" xyz="0.4385 0 0.387"/>
+  <!-- 0.387 -->
   <gazebo>
     <plugin name="gazebo_ros_control" filename="libgazebo_ros_control.so">
-      <robotNamespace>/msd_tunnel_dtw</robotNamespace>
+      <robotNamespace>/msd_tunnel_sensor</robotNamespace>
       <robotSimType>gazebo_ros_control/DefaultRobotHWSim</robotSimType>
       <legacyModeNS>true</legacyModeNS>
