Commit message: change directory structure

File: xacro/msd_tunnel_sensor.xacro (robot description, xacro)
@@ -30,5 +30,5 @@
       <visual>
         <geometry>
-          <mesh filename="package://msd_simulator/model/meshes/msd_tunnel/drive_wheel.dae"/>
+          <mesh filename="package://msd_simulator/model/msd_tunnel/meshes/drive_wheel.dae"/>
         </geometry>
         <material name="red"/>
@@ -63,5 +63,5 @@
         <origin xyz="0 0 0" rpy="0 0 0" />
         <geometry>
-          <mesh filename="package://msd_simulator/model/meshes/msd_tunnel/roller.dae" />
+          <mesh filename="package://msd_simulator/model/msd_tunnel/meshes/roller.dae" />
         </geometry>
       </visual>
@@ -94,5 +94,5 @@
         </geometry> -->
         <geometry>
-          <mesh filename="package://msd_simulator/model/meshes/msd_tunnel/rplidar-s1m1-r1.dae"/>
+          <mesh filename="package://msd_simulator/model/msd_tunnel/meshes/rplidar-s1m1-r1.dae"/>
         </geometry>
         <material name="red" />
@@ -104,5 +104,5 @@
         </geometry> -->
         <geometry>
-          <mesh filename="package://msd_simulator/model/meshes/msd_tunnel/rplidar-s1m1-r1.dae"/>
+          <mesh filename="package://msd_simulator/model/meshes/rplidar-s1m1-r1.dae"/>
         </geometry>
       </collision>
@@ -157,5 +157,5 @@
       <origin xyz="0 0 0" rpy="0 0 0" />
       <geometry>
-        <mesh filename="package://msd_simulator/model/meshes/msd_tunnel/body.dae" />
+        <mesh filename="package://msd_simulator/model/msd_tunnel/meshes/body.dae" />
       </geometry>
       <material name="gray" />

Commit message: fix xacro dae filepath

File: xacro/msd_tunnel_sensor.xacro (robot description, xacro)
@@ -30,5 +30,5 @@
       <visual>
         <geometry>
-          <mesh filename="package://msd_simulator/model/msd_tunnel/meshes/drive_wheel.dae"/>
+          <mesh filename="package://msd_simulator/models/msd_tunnel/meshes/drive_wheel.dae"/>
         </geometry>
         <material name="red"/>
@@ -63,5 +63,5 @@
         <origin xyz="0 0 0" rpy="0 0 0" />
         <geometry>
-          <mesh filename="package://msd_simulator/model/msd_tunnel/meshes/roller.dae" />
+          <mesh filename="package://msd_simulator/models/msd_tunnel/meshes/roller.dae" />
         </geometry>
       </visual>
@@ -94,5 +94,5 @@
         </geometry> -->
         <geometry>
-          <mesh filename="package://msd_simulator/model/msd_tunnel/meshes/rplidar-s1m1-r1.dae"/>
+          <mesh filename="package://msd_simulator/models/msd_tunnel/meshes/rplidar-s1m1-r1.dae"/>
         </geometry>
         <material name="red" />
@@ -104,5 +104,5 @@
         </geometry> -->
         <geometry>
-          <mesh filename="package://msd_simulator/model/meshes/rplidar-s1m1-r1.dae"/>
+          <mesh filename="package://msd_simulator/models/msd_tunnel/meshes/rplidar-s1m1-r1.dae"/>
         </geometry>
       </collision>
@@ -157,5 +157,5 @@
       <origin xyz="0 0 0" rpy="0 0 0" />
       <geometry>
-        <mesh filename="package://msd_simulator/model/msd_tunnel/meshes/body.dae" />
+        <mesh filename="package://msd_simulator/models/msd_tunnel/meshes/body.dae" />
       </geometry>
       <material name="gray" />
